Commit message: done

File: output.urdf (robot description, URDF)
Before this commit: robot xarm7_robot, 17 links, 16 joints
Links:
- link link1: geometry collision mesh filename=meshes/link1.stl; visual mesh filename=meshes/link1.stl
- link link2: geometry collision mesh filename=meshes/link2.stl; visual mesh filename=meshes/link2.stl
- link link3: geometry collision mesh filename=meshes/link3.stl; visual mesh filename=meshes/link3.stl
- link link4: geometry collision mesh filename=meshes/link4.stl; visual mesh filename=meshes/link4.stl
- link link5: geometry collision mesh filename=meshes/link5.stl; visual mesh filename=meshes/link5.stl
- link link6: geometry collision mesh filename=meshes/link6.stl; visual mesh filename=meshes/link6.stl
- link link7: geometry collision mesh filename=meshes/link7.stl; visual mesh filename=meshes/link7.stl
- link link_base: geometry collision mesh filename=meshes/link_base.stl; visual mesh filename=meshes/link_base.stl
